Commit message: gazebo simulation with controls

File: description/robot.urdf.xacro (robot description, xacro)
@@ -2,3 +2,4 @@
 <robot xmlns:xacro="http://www.ros.org/wiki/xacro"  name="robot">
     <xacro:include filename="robot_st.xacro" />
+    <xacro:include filename="gazebo_control.xacro" />
 </robot>

File: description/robot_st.xacro (robot description, xacro)
@@ -44,4 +44,7 @@
         </xacro:inertial_box>
     </link>
+    <gazebo reference="robot_body">
+        <material>Gazebo/Yellow</material>
+    </gazebo>
     <!-- Robot's front axis -->
     <link name="front_axis">
@@ -57,4 +60,7 @@
         </xacro:inertial_cylinder>
     </link>
+    <gazebo reference="front_axis">
+         <material>Gazebo/Black</material>
+    </gazebo>
     <joint name="axis_joint_front" type="fixed">
         <parent link="robot_body"/>
@@ -75,4 +81,7 @@
         </xacro:inertial_cylinder>
     </link>
+    <gazebo reference="rear_axis">
+         <material>Gazebo/Black</material>
+     </gazebo>
     <joint name="axis_joint_rear" type="fixed">
         <parent link="robot_body"/>
@@ -82,4 +91,26 @@
     <!-- Front axis wheels-->
     <!--wheel 1-->
+    <link name="front_right_wheel">
+        <visual>
+            <geometry><cylinder radius="0.05" length="0.02"/></geometry> <!-- wheel size-->
+            <material name="black"/>
+        </visual>
+        <collision>
+            <geometry><cylinder radius="0.05" length="0.02"/></geometry> <!-- wheel size-->
+        </collision>
+        <xacro:inertial_cylinder mass="0.03" length="0.2" radius="0.05"> <!--wheel inertia-->
+            <origin xyz="0 0 0" rpy="0 0 0"/>
+        </xacro:inertial_cylinder>
+    </link>
+    <gazebo reference="front_right_wheel">
+        <material>Gazebo/Black</material>
+    </gazebo>
+    <joint name="front_right_wheel_joint" type="continuous"> <!--Needs to be continuous for movement  (fixed for RVIZ2 setup)-->
+        <parent link="front_axis"/>
+        <child link="front_right_wheel"/>
+        <origin xyz="0 0 0.175" rpy="0 0 0"/>
+        <axis xyz="0 0 1"/> <!-- axis of rotation for the wheel -->
+    </joint>
+    <!--wheel 2-->
     <link name="front_left_wheel">
         <visual>
@@ -94,29 +125,37 @@
         </xacro:inertial_cylinder>
     </link>
+    <gazebo reference="front_left_wheel">
+        <material>Gazebo/Black</material>
+    </gazebo>
     <joint name="front_left_wheel_joint" type="continuous"> <!--Needs to be continuous for movement  (fixed for RVIZ2 setup)-->
         <parent link="front_axis"/>
         <child link="front_left_wheel"/>
-        <origin xyz="0 0 0.175" rpy="0 0 0"/>
-    </joint>
-    <!--wheel 2-->
-    <link name="front_right_wheel">
-        <visual>
-            <geometry><cylinder radius="0.05" length="0.02"/></geometry> <!-- wheel size-->
-            <material name="black"/>
-        </visual>
-        <collision>
-            <geometry><cylinder radius="0.05" length="0.02"/></geometry> <!-- wheel size-->
-        </collision>
-        <xacro:inertial_cylinder mass="0.03" length="0.2" radius="0.05"> <!--wheel inertia-->
-            <origin xyz="0 0 0" rpy="0 0 0"/>
-        </xacro:inertial_cylinder>
-    </link>
-    <joint name="front_right_wheel_joint" type="continuous"> <!--Needs to be continuous for movement  (fixed for RVIZ2 setup)-->
-        <parent link="front_axis"/>
-        <child link="front_right_wheel"/>
         <origin xyz="0 0 -0.175" rpy="0 0 0"/>
+        <axis xyz="0 0 1"/> <!-- axis of rotation for the wheel -->
     </joint>
 <!-- rear axis wheels-->
     <!--wheel 1-->
+    <link name="rear_right_wheel">
+        <visual>
+            <geometry><cylinder radius="0.05" length="0.02"/></geometry> <!-- wheel size-->
+            <material name="black"/>
+        </visual>
+        <collision>
+            <geometry><cylinder radius="0.05" length="0.02"/></geometry> <!-- wheel size-->
+        </collision>
+        <xacro:inertial_cylinder mass="0.03" length="0.2" radius="0.05"> <!--wheel inertia-->
+            <origin xyz="0 0 0" rpy="0 0 0"/>
+        </xacro:inertial_cylinder>
+    </link>
+    <gazebo reference="rear_right_wheel">
+         <material>Gazebo/Black</material>
+    </gazebo>
+    <joint name="rear_right_wheel_joint" type="continuous"> <!--Needs to be continuous for movement  (fixed for RVIZ2 setup)-->
+        <parent link="rear_axis"/>
+        <child link="rear_right_wheel"/>
+        <origin xyz="0 0 0.175" rpy="0 0 0"/>
+        <axis xyz="0 0 1"/> <!-- axis of rotation for the wheel -->
+    </joint>
+    <!--wheel 2-->
     <link name="rear_left_wheel">
         <visual>
@@ -131,26 +170,12 @@
         </xacro:inertial_cylinder>
     </link>
+    <gazebo reference="rear_left_wheel">
+        <material>Gazebo/Black</material>
+    </gazebo>
     <joint name="rear_left_wheel_joint" type="continuous"> <!--Needs to be continuous for movement  (fixed for RVIZ2 setup)-->
         <parent link="rear_axis"/>
         <child link="rear_left_wheel"/>
-        <origin xyz="0 0 0.175" rpy="0 0 0"/>
-    </joint>
-    <!--wheel 2-->
-    <link name="rear_right_wheel">
-        <visual>
-            <geometry><cylinder radius="0.05" length="0.02"/></geometry> <!-- wheel size-->
-            <material name="black"/>
-        </visual>
-        <collision>
-            <geometry><cylinder radius="0.05" length="0.02"/></geometry> <!-- wheel size-->
-        </collision>
-        <xacro:inertial_cylinder mass="0.03" length="0.2" radius="0.05"> <!--wheel inertia-->
-            <origin xyz="0 0 0" rpy="0 0 0"/>
-        </xacro:inertial_cylinder>
-    </link>
-    <joint name="rear_right_wheel_joint" type="continuous"> <!--Needs to be continuous for movement  (fixed for RVIZ2 setup)-->
-        <parent link="rear_axis"/>
-        <child link="rear_right_wheel"/>
         <origin xyz="0 0 -0.175" rpy="0 0 0"/>
+        <axis xyz="0 0 1"/> <!-- axis of rotation for the wheel -->
     </joint>
     <!-- Robot's depth camera -->
@@ -167,4 +192,7 @@
         </xacro:inertial_box>
     </link>
+     <gazebo reference="camera_link">
+        <material>Gazebo/Black</material>
+    </gazebo>
     <joint name="camera_joint" type="fixed">
         <parent link="robot_body"/>
