Commit message: Add grey material definition to robot RViz colors

File: description/robot_rviz_colors.xacro (robot description, xacro)
@@ -20,3 +20,6 @@
         <color rgba="1 1 0 0.5"/>
     </material>
+    <material name="grey">
+        <color rgba="0.5 0.5 0.5 1"/>
+    </material>
 </robot>
