Commit message: wheel_type_continuous

File: description/robot_st.xacro (robot description, xacro)
@@ -67,5 +67,5 @@
         </visual>
     </link>
-    <joint name="front_left_wheel_joint" type="fixed"> <!--Needs to be continuous for movement  (fixed for RVIZ2 setup)-->
+    <joint name="front_left_wheel_joint" type="continuous"> <!--Needs to be continuous for movement  (fixed for RVIZ2 setup)-->
         <parent link="front_axis"/>
         <child link="front_left_wheel"/>
@@ -79,5 +79,5 @@
         </visual>
     </link>
-    <joint name="front_right_wheel_joint" type="fixed"> <!--Needs to be continuous for movement  (fixed for RVIZ2 setup)-->
+    <joint name="front_right_wheel_joint" type="continuous"> <!--Needs to be continuous for movement  (fixed for RVIZ2 setup)-->
         <parent link="front_axis"/>
         <child link="front_right_wheel"/>
@@ -92,5 +92,5 @@
         </visual>
     </link>
-    <joint name="rear_left_wheel_joint" type="fixed"> <!--Needs to be continuous for movement  (fixed for RVIZ2 setup)-->
+    <joint name="rear_left_wheel_joint" type="continuous"> <!--Needs to be continuous for movement  (fixed for RVIZ2 setup)-->
         <parent link="rear_axis"/>
         <child link="rear_left_wheel"/>
@@ -104,5 +104,5 @@
         </visual>
     </link>
-    <joint name="rear_right_wheel_joint" type="fixed"> <!--Needs to be continuous for movement  (fixed for RVIZ2 setup)-->
+    <joint name="rear_right_wheel_joint" type="continuous"> <!--Needs to be continuous for movement  (fixed for RVIZ2 setup)-->
         <parent link="rear_axis"/>
         <child link="rear_right_wheel"/>
@@ -119,5 +119,5 @@
         <parent link="robot_body"/>
         <child link="camera_link"/>
-        <origin xyz="0.15 0 0.1" rpy="0 0 0"/> <!-- XYZ to move RPY to rotate-->
+        <origin xyz="0.3 0 0.1" rpy="0 0 0"/> <!-- XYZ to move RPY to rotate-->
     </joint>
 </robot>

Commit message: Inertia properties

File: description/robot_st.xacro (robot description, xacro)
@@ -1,4 +1,5 @@
 <?xml version="1.0"?>
 <robot xmlns:xacro="http://www.ros.org/wiki/xacro">
+    <xacro:include filename="robot_inertia.xacro" />
     <!-- Color library -->
     <material name="black">
@@ -34,4 +35,12 @@
             <material name="yellow"/>
         </visual>
+        <collision>
+            <geometry>
+                <box size="0.7 0.35 0.1"/> <!-- X-Y-Z robot's body (urdf's default in meters)-->
+            </geometry>
+        </collision>
+        <xacro:inertial_box mass="1.0" x="0.7" y="0.35" z="0.1"> <!--Main body inertia-->
+            <origin xyz="0 0 0" rpy="0 0 0"/>
+        </xacro:inertial_box>
     </link>
     <!-- Robot's front axis -->
@@ -41,4 +50,10 @@
             <material name="black"/>
         </visual>
+        <collision>
+            <geometry><cylinder radius="0.005" length="0.35"/></geometry> <!-- axis size-->
+        </collision>
+        <xacro:inertial_cylinder mass="0.01" length="0.35" radius="0.005"> <!--Wheel/axis inertia-->
+            <origin xyz="0 0 0" rpy="0 0 0"/>
+        </xacro:inertial_cylinder>
     </link>
     <joint name="axis_joint_front" type="fixed">
@@ -53,4 +68,10 @@
             <material name="black"/>
         </visual>
+        <collision>
+            <geometry><cylinder radius="0.005" length="0.35"/></geometry> <!-- axis size-->
+        </collision>
+        <xacro:inertial_cylinder mass="0.01" length="0.35" radius="0.005"> <!--axis inertia-->
+            <origin xyz="0 0 0" rpy="0 0 0"/>
+        </xacro:inertial_cylinder>
     </link>
     <joint name="axis_joint_rear" type="fixed">
@@ -66,4 +87,10 @@
             <material name="black"/>
         </visual>
+        <collision>
+            <geometry><cylinder radius="0.05" length="0.02"/></geometry> <!-- wheel size-->
+        </collision>
+        <xacro:inertial_cylinder mass="0.03" length="0.2" radius="0.05"> <!--wheel inertia-->
+            <origin xyz="0 0 0" rpy="0 0 0"/>
+        </xacro:inertial_cylinder>
     </link>
     <joint name="front_left_wheel_joint" type="continuous"> <!--Needs to be continuous for movement  (fixed for RVIZ2 setup)-->
@@ -78,4 +105,10 @@
             <material name="black"/>
         </visual>
+        <collision>
+            <geometry><cylinder radius="0.05" length="0.02"/></geometry> <!-- wheel size-->
+        </collision>
+        <xacro:inertial_cylinder mass="0.03" length="0.2" radius="0.05"> <!--wheel inertia-->
+            <origin xyz="0 0 0" rpy="0 0 0"/>
+        </xacro:inertial_cylinder>
     </link>
     <joint name="front_right_wheel_joint" type="continuous"> <!--Needs to be continuous for movement  (fixed for RVIZ2 setup)-->
@@ -91,4 +124,10 @@
             <material name="black"/>
         </visual>
+        <collision>
+            <geometry><cylinder radius="0.05" length="0.02"/></geometry> <!-- wheel size-->
+        </collision>
+        <xacro:inertial_cylinder mass="0.03" length="0.2" radius="0.05"> <!--wheel inertia-->
+            <origin xyz="0 0 0" rpy="0 0 0"/>
+        </xacro:inertial_cylinder>
     </link>
     <joint name="rear_left_wheel_joint" type="continuous"> <!--Needs to be continuous for movement  (fixed for RVIZ2 setup)-->
@@ -103,4 +142,10 @@
             <material name="black"/>
         </visual>
+        <collision>
+            <geometry><cylinder radius="0.05" length="0.02"/></geometry> <!-- wheel size-->
+        </collision>
+        <xacro:inertial_cylinder mass="0.03" length="0.2" radius="0.05"> <!--wheel inertia-->
+            <origin xyz="0 0 0" rpy="0 0 0"/>
+        </xacro:inertial_cylinder>
     </link>
     <joint name="rear_right_wheel_joint" type="continuous"> <!--Needs to be continuous for movement  (fixed for RVIZ2 setup)-->
@@ -115,4 +160,10 @@
             <material name="black"/>
         </visual>
+        <collision>
+            <geometry><box size="0.05 0.15 0.1"/></geometry> <!-- camera size-->
+        </collision>
+        <xacro:inertial_box mass="0.1" x="0.05" y="0.15" z="0.1"> <!--camera inertia-->
+            <origin xyz="0 0 0" rpy="0 0 0"/>
+        </xacro:inertial_box>
     </link>
     <joint name="camera_joint" type="fixed">

Commit message: Remove color materials from robot_st.xacro
Removed color material definitions from the robot description file.

File: description/robot_st.xacro (robot description, xacro)
@@ -2,23 +2,5 @@
 <robot xmlns:xacro="http://www.ros.org/wiki/xacro">
     <xacro:include filename="robot_inertia.xacro" />
-    <!-- Color library -->
-    <material name="black">
-        <color rgba="0 0 0 1"/>
-    </material>
-    <material name="white">
-        <color rgba="1 1 1 1"/>
-    </material>
-    <material name="red">
-        <color rgba="1 0 0 1"/>
-    </material>
-    <material name="green">
-        <color rgba="0 1 0 1"/>
-    </material>
-    <material name="blue">
-        <color rgba="0 0 1 1"/>
-    </material>
-    <material name="yellow">
-        <color rgba="1 1 0 0.5"/>
-    </material>
+    <xacro:include filename="robot_rviz_colors" />
     <!-- Base link, needed due to some limitations in rviz2 -->
     <link name="base_link"/>

Commit message: Refactor robot parameters and add wheel macros
Updated robot parameters and dimensions in robot_st.xacro to use properties for body, wheels, and camera. Introduced macros for wheel creation and adjusted joint origins for axes.

File: description/robot_st.xacro (robot description, xacro)
@@ -3,6 +3,29 @@
     <xacro:include filename="robot_inertia.xacro" />
     <xacro:include filename="robot_rviz_colors" />
+    <!-- ========================================= -->
+    <!-- Robot parameters - change here -->
+    <!-- ========================================= -->
+    <!-- Main body -->
+    <xacro:property name="body_length" value="0.7" />    <!-- (X) -->
+    <xacro:property name="body_width" value="0.35" />  <!-- (Y) -->
+    <xacro:property name="body_height" value="0.1" />    <!-- (Z) -->
+    <xacro:property name="body_mass" value="1.0" />
+    <!-- Axes -->
+    <xacro:property name="axis_radius" value="0.005" />
+    <xacro:property name="axis_mass" value="0.01" />
+    <!-- Wheels -->
+    <xacro:property name="wheel_radius" value="0.05" />
+    <xacro:property name="wheel_width" value="0.02" />
+    <xacro:property name="wheel_mass" value="0.03" />
+    <!-- camera (relative to other dimensions) -->
+    <xacro:property name="camera_size_x" value="0.05" />
+    <xacro:property name="camera_size_y" value="${body_width * 0.5}" />  <!-- half main body width -->
+    <xacro:property name="camera_size_z" value="0.1" />
+    <xacro:property name="camera_mass" value="0.1" />
+    <!-- Distance from center  (wheel base / 2) -->
+    <xacro:property name="wheel_base_half" value="${body_length * 0.35}" />  <!-- 35% from length -->
+    <xacro:property name="axis_height" value="${body_height * 0.5 + wheel_radius}" />
     <!-- Base link, needed due to some limitations in rviz2 -->
-    <link name="base_link"/>
+link name="base_link"/>
     <joint name="base_to_body" type="fixed">
         <parent link="base_link"/>
@@ -13,5 +36,5 @@
         <visual>
             <geometry>
-                <box size="0.7 0.35 0.1"/> <!-- X-Y-Z robot's body (urdf's default in meters)-->
+                <box size="${body_length} ${body_width} ${body_height}"/>
             </geometry>
             <material name="yellow"/>
@@ -19,8 +42,8 @@
         <collision>
             <geometry>
-                <box size="0.7 0.35 0.1"/> <!-- X-Y-Z robot's body (urdf's default in meters)-->
+                <box size="${body_length} ${body_width} ${body_height}"/>
             </geometry>
         </collision>
-        <xacro:inertial_box mass="1.0" x="0.7" y="0.35" z="0.1"> <!--Main body inertia-->
+        <xacro:inertial_box mass="${body_mass}" x="${body_length}" y="${body_width}" z="${body_height}">
             <origin xyz="0 0 0" rpy="0 0 0"/>
         </xacro:inertial_box>
@@ -29,150 +52,87 @@
         <material>Gazebo/Yellow</material>
     </gazebo>
-    <!-- Robot's front axis -->
-    <link name="front_axis">
+    <!-- ========================================= -->
+    <!-- Axes (front and rear) -->
+    <!-- ========================================= -->
+    <!-- Axes -->
+    <xacro:macro name="wheel_axis" params="name">
+        <link name="${name}_axis">
+            <visual>
+                <geometry><cylinder radius="${axis_radius}" length="${body_width}"/></geometry>
+                <material name="black"/>
+            </visual>
+            <collision>
+                <geometry><cylinder radius="${axis_radius}" length="${body_width}"/></geometry>
+            </collision>
+            <xacro:inertial_cylinder mass="${axis_mass}" length="${body_width}" radius="${axis_radius}">
+                <origin xyz="0 0 0" rpy="0 0 0"/>
+            </xacro:inertial_cylinder>
+        </link>
+        <gazebo reference="${name}_axis">
+            <material>Gazebo/Black</material>
+        </gazebo>
+    </xacro:macro>
+    <!-- create axes -->
+    <xacro:wheel_axis name="front"/>
+    <xacro:wheel_axis name="rear"/>
+    <!-- axes and body joints -->
+    <joint name="axis_joint_front" type="fixed">
+        <parent link="robot_body"/>
+        <child link="front_axis"/>
+        <origin xyz="${wheel_base_half} 0 ${-axis_height}" rpy="${pi/2} 0 0"/>
+    </joint>
+    <joint name="axis_joint_rear" type="fixed">
+        <parent link="robot_body"/>
+        <child link="rear_axis"/>
+        <origin xyz="${-wheel_base_half} 0 ${-axis_height}" rpy="${pi/2} 0 0"/>
+    </joint>
+    <!-- ========================================= -->
+    <!-- Wheels (macro) -->
+    <!-- ========================================= -->
+    <xacro:macro name="wheel" params="name parent side">
+        <!-- side: 1 for right wheel, -1 for left wheel -->
+        <link name="${name}_wheel">
+            <visual>
+                <geometry><cylinder radius="${wheel_radius}" length="${wheel_width}"/></geometry>
+                <material name="black"/>
+            </visual>
+            <collision>
+                <geometry><cylinder radius="${wheel_radius}" length="${wheel_width}"/></geometry>
+            </collision>
+            <xacro:inertial_cylinder mass="${wheel_mass}" length="${wheel_width}" radius="${wheel_radius}">
+                <origin xyz="0 0 0" rpy="0 0 0"/>
+            </xacro:inertial_cylinder>
+        </link>
+        <gazebo reference="${name}_wheel">
+            <material>Gazebo/Black</material>
+        </gazebo>
+        <joint name="${name}_wheel_joint" type="continuous">
+            <parent link="${parent}_axis"/>
+            <child link="${name}_wheel"/>
+            <origin xyz="0 0 ${side * (body_width/2)}" rpy="0 0 0"/>
+            <axis xyz="0 0 1"/>
+        </joint>
+    </xacro:macro>
+    <!-- 4 wheels -->
+    <xacro:wheel name="front_right" parent="front" side="1"/>
+    <xacro:wheel name="front_left" parent="front" side="-1"/>
+    <xacro:wheel name="rear_right" parent="rear" side="1"/>
+    <xacro:wheel name="rear_left" parent="rear" side="-1"/>
+    <!-- ========================================= -->
+    <!-- Camera -->
+    <!-- ========================================= -->
+    <link name="camera_link">
         <visual>
-            <geometry><cylinder radius="0.005" length="0.35"/></geometry> <!-- axis size-->
+            <geometry><box size="${camera_size_x} ${camera_size_y} ${camera_size_z}"/></geometry>
             <material name="black"/>
         </visual>
         <collision>
-            <geometry><cylinder radius="0.005" length="0.35"/></geometry> <!-- axis size-->
+            <geometry><box size="${camera_size_x} ${camera_size_y} ${camera_size_z}"/></geometry>
         </collision>
-        <xacro:inertial_cylinder mass="0.01" length="0.35" radius="0.005"> <!--Wheel/axis inertia-->
-            <origin xyz="0 0 0" rpy="0 0 0"/>
-        </xacro:inertial_cylinder>
-    </link>
-    <gazebo reference="front_axis">
-         <material>Gazebo/Black</material>
-    </gazebo>
-    <joint name="axis_joint_front" type="fixed">
-        <parent link="robot_body"/>
-        <child link="front_axis"/>
-        <origin xyz="0.25 0 -0.05" rpy="${pi/2} 0 0"/> <!-- XYZ to move RPY to rotate-->
-    </joint>
-    <!-- Robot's rear axis -->
-    <link name="rear_axis">
-        <visual>
-            <geometry><cylinder radius="0.005" length="0.35"/></geometry> <!-- axis size-->
-            <material name="black"/>
-        </visual>
-        <collision>
-            <geometry><cylinder radius="0.005" length="0.35"/></geometry> <!-- axis size-->
-        </collision>
-        <xacro:inertial_cylinder mass="0.01" length="0.35" radius="0.005"> <!--axis inertia-->
-            <origin xyz="0 0 0" rpy="0 0 0"/>
-        </xacro:inertial_cylinder>
-    </link>
-    <gazebo reference="rear_axis">
-         <material>Gazebo/Black</material>
-     </gazebo>
-    <joint name="axis_joint_rear" type="fixed">
-        <parent link="robot_body"/>
-        <child link="rear_axis"/>
-        <origin xyz="-0.25 0 -0.05" rpy="${pi/2} 0 0"/> <!-- XYZ to move RPY to rotate-->
-    </joint>
-    <!-- Front axis wheels-->
-    <!--wheel 1-->
-    <link name="front_right_wheel">
-        <visual>
-            <geometry><cylinder radius="0.05" length="0.02"/></geometry> <!-- wheel size-->
-            <material name="black"/>
-        </visual>
-        <collision>
-            <geometry><cylinder radius="0.05" length="0.02"/></geometry> <!-- wheel size-->
-        </collision>
-        <xacro:inertial_cylinder mass="0.03" length="0.2" radius="0.05"> <!--wheel inertia-->
-            <origin xyz="0 0 0" rpy="0 0 0"/>
-        </xacro:inertial_cylinder>
-    </link>
-    <gazebo reference="front_right_wheel">
-        <material>Gazebo/Black</material>
-    </gazebo>
-    <joint name="front_right_wheel_joint" type="continuous"> <!--Needs to be continuous for movement  (fixed for RVIZ2 setup)-->
-        <parent link="front_axis"/>
-        <child link="front_right_wheel"/>
-        <origin xyz="0 0 0.175" rpy="0 0 0"/>
-        <axis xyz="0 0 1"/> <!-- axis of rotation for the wheel -->
-    </joint>
-    <!--wheel 2-->
-    <link name="front_left_wheel">
-        <visual>
-            <geometry><cylinder radius="0.05" length="0.02"/></geometry> <!-- wheel size-->
-            <material name="black"/>
-        </visual>
-        <collision>
-            <geometry><cylinder radius="0.05" length="0.02"/></geometry> <!-- wheel size-->
-        </collision>
-        <xacro:inertial_cylinder mass="0.03" length="0.2" radius="0.05"> <!--wheel inertia-->
-            <origin xyz="0 0 0" rpy="0 0 0"/>
-        </xacro:inertial_cylinder>
-    </link>
-    <gazebo reference="front_left_wheel">
-        <material>Gazebo/Black</material>
-    </gazebo>
-    <joint name="front_left_wheel_joint" type="continuous"> <!--Needs to be continuous for movement  (fixed for RVIZ2 setup)-->
-        <parent link="front_axis"/>
-        <child link="front_left_wheel"/>
-        <origin xyz="0 0 -0.175" rpy="0 0 0"/>
-        <axis xyz="0 0 1"/> <!-- axis of rotation for the wheel -->
-    </joint>
-<!-- rear axis wheels-->
-    <!--wheel 1-->
-    <link name="rear_right_wheel">
-        <visual>
-            <geometry><cylinder radius="0.05" length="0.02"/></geometry> <!-- wheel size-->
-            <material name="black"/>
-        </visual>
-        <collision>
-            <geometry><cylinder radius="0.05" length="0.02"/></geometry> <!-- wheel size-->
-        </collision>
-        <xacro:inertial_cylinder mass="0.03" length="0.2" radius="0.05"> <!--wheel inertia-->
-            <origin xyz="0 0 0" rpy="0 0 0"/>
-        </xacro:inertial_cylinder>
-    </link>
-    <gazebo reference="rear_right_wheel">
-         <material>Gazebo/Black</material>
-    </gazebo>
-    <joint name="rear_right_wheel_joint" type="continuous"> <!--Needs to be continuous for movement  (fixed for RVIZ2 setup)-->
-        <parent link="rear_axis"/>
-        <child link="rear_right_wheel"/>
-        <origin xyz="0 0 0.175" rpy="0 0 0"/>
-        <axis xyz="0 0 1"/> <!-- axis of rotation for the wheel -->
-    </joint>
-    <!--wheel 2-->
-    <link name="rear_left_wheel">
-        <visual>
-            <geometry><cylinder radius="0.05" length="0.02"/></geometry> <!-- wheel size-->
-            <material name="black"/>
-        </visual>
-        <collision>
-            <geometry><cylinder radius="0.05" length="0.02"/></geometry> <!-- wheel size-->
-        </collision>
-        <xacro:inertial_cylinder mass="0.03" length="0.2" radius="0.05"> <!--wheel inertia-->
-            <origin xyz="0 0 0" rpy="0 0 0"/>
-        </xacro:inertial_cylinder>
-    </link>
-    <gazebo reference="rear_left_wheel">
-        <material>Gazebo/Black</material>
-    </gazebo>
-    <joint name="rear_left_wheel_joint" type="continuous"> <!--Needs to be continuous for movement  (fixed for RVIZ2 setup)-->
-        <parent link="rear_axis"/>
-        <child link="rear_left_wheel"/>
-        <origin xyz="0 0 -0.175" rpy="0 0 0"/>
-        <axis xyz="0 0 1"/> <!-- axis of rotation for the wheel -->
-    </joint>
-    <!-- Robot's depth camera -->
-    <link name="camera_link">
-        <visual>
-            <geometry><box size="0.05 0.15 0.1"/></geometry> <!-- camera size-->
-            <material name="black"/>
-        </visual>
-        <collision>
-            <geometry><box size="0.05 0.15 0.1"/></geometry> <!-- camera size-->
-        </collision>
-        <xacro:inertial_box mass="0.1" x="0.05" y="0.15" z="0.1"> <!--camera inertia-->
+        <xacro:inertial_box mass="${camera_mass}" x="${camera_size_x}" y="${camera_size_y}" z="${camera_size_z}">
             <origin xyz="0 0 0" rpy="0 0 0"/>
         </xacro:inertial_box>
     </link>
-     <gazebo reference="camera_link">
+    <gazebo reference="camera_link">
         <material>Gazebo/Black</material>
     </gazebo>
@@ -180,5 +140,5 @@
         <parent link="robot_body"/>
         <child link="camera_link"/>
-        <origin xyz="0.3 0 0.1" rpy="0 0 0"/> <!-- XYZ to move RPY to rotate-->
+        <origin xyz="${body_length/2} 0 ${body_height/2 + camera_size_z/2}" rpy="0 0 0"/>
     </joint>
 </robot>
